Commit message: gripper starts to show life

File: urdf/stompy_new/multiarm.urdf (robot description, URDF)
Before this commit: robot upper_limb_assembly_5_dof, 20 links, 19 joints
Joints:
- joint joint_full_arm_5_dof_1_lower_arm_1_dof_1_hand_1_slider_1: axis 0 0 -1 -> 0 0 1; limit lower=0.02 upper=0.03 effort=6 velocity=5 -> lower=-0.05 upper=0.0 effort=6 velocity=5; type fixed -> prismatic
- joint joint_full_arm_5_dof_1_lower_arm_1_dof_1_hand_1_slider_2: limit lower=0.01 upper=.03 effort=6 velocity=5 -> lower=0.0 upper=.05 effort=80 velocity=5; type fixed -> prismatic
- joint joint_full_arm_5_dof_2_lower_arm_1_dof_1_hand_1_slider_1: limit lower=0 upper=0.051 effort=6 velocity=5 -> lower=-0.05 upper=0. effort=80 velocity=5
- joint joint_full_arm_5_dof_2_lower_arm_1_dof_1_hand_1_slider_2: limit lower=-0.051 upper=0 effort=6 velocity=5 -> lower=-0.05 upper=0 effort=6 velocity=5
