Commit message: updates to all files, removing pasta

File: urdf/stompy/meshes/upper_limb_assembly_5_dof_merged_simplified.urdf (robot description, URDF)
Before this commit: robot upper_limb_assembly_5_dof, 18 links, 17 joints
Joints:
- joint joint_full_arm_5_dof_1_lower_arm_1_dof_1_hand_1_rmd_x4_24_mock_1_dof_x4: type fixed -> revolute
- joint joint_full_arm_5_dof_1_lower_arm_1_dof_1_hand_1_slider_1: type fixed -> revolute
- joint joint_full_arm_5_dof_1_lower_arm_1_dof_1_hand_1_slider_2: mimic (none) -> joint=joint_full_arm_5_dof_1_lower_arm_1_dof_1_hand_1_slider_1 multiplier=1 offset=0; type fixed -> revolute
- joint joint_full_arm_5_dof_2_lower_arm_1_dof_1_hand_1_rmd_x4_24_mock_1_dof_x4: type fixed -> revolute
- joint joint_full_arm_5_dof_2_lower_arm_1_dof_1_hand_1_slider_1: type fixed -> revolute
- joint joint_full_arm_5_dof_2_lower_arm_1_dof_1_hand_1_slider_2: mimic (none) -> joint=joint_full_arm_5_dof_2_lower_arm_1_dof_1_hand_1_slider_1 multiplier=1 offset=0; type fixed -> revolute
- joint joint_full_arm_5_dof_2_lower_arm_1_dof_1_rmd_x4_24_mock_2_dof_x4: type fixed -> revolute
- joint joint_full_arm_5_dof_2_upper_left_arm_1_rmd_x4_24_mock_1_dof_x4: type fixed -> revolute
- joint joint_full_arm_5_dof_2_upper_left_arm_1_rmd_x4_24_mock_2_dof_x4: type fixed -> revolute
- joint joint_full_arm_5_dof_2_upper_left_arm_1_rmd_x8_90_mock_1_dof_x8: type fixed -> revolute
- joint joint_full_arm_5_dof_2_upper_left_arm_1_rmd_x8_90_mock_2_dof_x8: type fixed -> revolute
- joint joint_torso_1_rmd_x8_90_mock_1_dof_x8: type fixed -> revolute

File: urdf/stompy/upper_limb_assembly_5_dof_merged_simplified.urdf (robot description, URDF)
Before this commit: robot upper_limb_assembly_5_dof, 20 links, 19 joints
Joints:
- joint joint_full_arm_5_dof_1_lower_arm_1_dof_1_hand_1_slider_1: axis 0 0 1 -> 0 0 -1; limit lower=-0.05 upper=0.0 effort=6 velocity=5 -> lower=0 upper=0.05 effort=6 velocity=5
- joint joint_full_arm_5_dof_1_lower_arm_1_dof_1_hand_1_slider_2: limit lower=0.0 upper=.05 effort=80 velocity=5 -> lower=0 upper=.05 effort=80 velocity=5
