Commit message: update to the second gripper

File: urdf/stompy/upper_limb_assembly_5_dof_merged_simplified.urdf (robot description, URDF)
Before this commit: robot upper_limb_assembly_5_dof, 20 links, 19 joints
Joints:
- joint joint_full_arm_5_dof_2_lower_arm_1_dof_1_hand_1_slider_1: type fixed -> prismatic
- joint joint_full_arm_5_dof_2_lower_arm_1_dof_1_hand_1_slider_2: type fixed -> prismatic

Commit message: update firmware and grippers

File: urdf/stompy/upper_limb_assembly_5_dof_merged_simplified.urdf (robot description, URDF)
Before this commit: robot upper_limb_assembly_5_dof, 20 links, 19 joints
Joints:
- joint joint_full_arm_5_dof_2_lower_arm_1_dof_1_hand_1_slider_1: limit lower=-0.05 upper=0. effort=80 velocity=5 -> lower=0 upper=0.05 effort=80 velocity=5
- joint joint_full_arm_5_dof_2_lower_arm_1_dof_1_hand_1_slider_2: limit lower=-0.05 upper=0 effort=6 velocity=5 -> lower=5 upper=0.05 effort=6 velocity=5

Commit message: update pasta fix urdf

File: urdf/stompy/upper_limb_assembly_5_dof_merged_simplified.urdf (robot description, URDF)
Before this commit: robot upper_limb_assembly_5_dof, 20 links, 19 joints
Joints:
- joint joint_full_arm_5_dof_2_lower_arm_1_dof_1_hand_1_slider_2: limit lower=5 upper=0.05 effort=6 velocity=5 -> lower=0 upper=0.05 effort=6 velocity=5

Commit message: adding new version of firmware

File: urdf/stompy/upper_limb_assembly_5_dof_merged_simplified.urdf (robot description, URDF)
Before this commit: robot upper_limb_assembly_5_dof, 20 links, 19 joints
Joints:
- joint joint_full_arm_5_dof_2_lower_arm_1_dof_1_hand_1_slider_1: type prismatic -> fixed
- joint joint_full_arm_5_dof_2_lower_arm_1_dof_1_hand_1_slider_2: type prismatic -> fixed
