Commit message: add end effectors and set up position

File: urdf/stompy_mini/full_assembly_simplified.urdf (robot description, URDF)
Before this commit: robot full_assembly, 253 links, 252 joints
Links:
- added link left_end_effector_link
- added link right_end_effector_link
Joints:
- added joint left_end_effector_joint: type fixed, parent link_upper_half_assembly_1_left_arm_1_robstride_01_mock_4_rs_01_rotor_1, child left_end_effector_link, origin xyz=-.05 0 -.1 rpy=0 0 0
- added joint right_end_effector_joint: type fixed, parent link_upper_half_assembly_1_right_arm_1_robstride_01_mock_4_rs_01_rotor_1, child right_end_effector_link, origin xyz=-.05 0 -.1 rpy=0 0 0
