Commit message: right arm responsive and properly working

File: urdf/stompy_mini/upper_half_assembly_simplified.urdf (robot description, URDF)
Before this commit: robot upper_half_assembly, 95 links, 94 joints
Joints:
- joint left elbow pitch: limit lower=-1.3089969 upper=1.8325957 effort=80 velocity=5 -> lower=-1.3089969 upper=1.8325957 effort=6 velocity=5; type revolute -> fixed
- joint left shoulder pitch: limit lower=0.034906585 upper=5.2185345 effort=80 velocity=5 -> lower=-4 upper=4 effort=6 velocity=5; type revolute -> fixed
- joint left shoulder roll: limit lower=-1.2740904 upper=1.8325957 effort=80 velocity=5 -> lower=-4.2740904 upper=-1.8325957 effort=6 velocity=5; type revolute -> fixed
- joint left shoulder yaw: limit lower=-1.3089969 upper=1.8762289 effort=80 velocity=5 -> lower=-3.3089969 upper=3.8762289 effort=6 velocity=5; type revolute -> fixed
- joint left wrist roll: limit lower=-3.1415927 upper=0 effort=80 velocity=5 -> lower=-3.1415927 upper=0 effort=6 velocity=5
- joint right elbow pitch: limit lower=1.8325957 upper=3.403392 effort=80 velocity=5 -> lower=0.8325957 upper=4.403392 effort=6 velocity=5
- joint right shoulder pitch: limit lower=-1.012291 upper=4.1538836 effort=80 velocity=5 -> lower=0.012291 upper=5.1538836 effort=6 velocity=5
- joint right shoulder roll: limit lower=-3.3684855 upper=-0.26179939 effort=80 velocity=5 -> lower=-3.3684855 upper=.26179939 effort=6 velocity=5
- joint right shoulder yaw: limit lower=-1.3089969 upper=1.8325957 effort=80 velocity=5 -> lower=-3.3089969 upper=1.2325957 effort=6 velocity=5
- joint right wrist roll: limit lower=-3.1415927 upper=3.1415927 effort=80 velocity=5 -> lower=-3.1415927 upper=3.1415927 effort=6 velocity=5
