Commit message: switch to torso

File: urdf/stompy_pro/robot.urdf (robot description, URDF)
Before this commit: robot robot, 22 links, 21 joints
Links:
- removed link L_buttock
- removed link L_calf
- removed link L_foot
- removed link L_leg
- removed link L_thigh
- removed link R_buttock
- removed link R_calf
- removed link R_foot
- removed link R_leg
- removed link R_thigh
Joints:
- removed joint L_ankle_y
- removed joint L_hip_x
- removed joint L_hip_y
- removed joint L_hip_z
- removed joint L_knee
- removed joint R_ankle_y
- removed joint R_hip_x
- removed joint R_hip_y
- removed joint R_hip_z
- removed joint R_knee
